Commit message: fix issue with controllers

File: robot_description_simulation/robots/rbkairos/rbkairos_ur.urdf.xacro (robot description, xacro)
@@ -5,7 +5,23 @@
   <!-- ***************** -->
   <!-- First we import all posible elements defined in the urdf.xacro files. All these elements are defined as macro:xacros -->
+  <xacro:arg name="controllers" default="$(find robotnik_gazebo_classic)/config/rbkairos_control_gazebo.yaml"/>
   <xacro:include filename="$(find robot_description)/macros/rbkairos_macro.urdf.xacro" />
   <xacro:include filename="$(find robot_description_simulation)/ros2_control/classic/rbkairos_control.urdf.xacro"/>
   <xacro:include filename="$(find robot_description_simulation)/ros2_control/ignition/rbkairos_control.urdf.xacro"/>
+  <!-- Import UR arm -->
+  <!-- <xacro:include filename="$(find ur_description)/urdf/ur.urdf.xacro" /> -->
+  <xacro:arg name="ur_type" default="ur5e"/>
+  <xacro:arg name="name" default="$(arg ur_type)"/>
+  <xacro:arg name="prefix" default="rbkairos_"/>
+  <xacro:arg name="joint_limit_params" default="$(find ur_description)/config/$(arg ur_type)/joint_limits.yaml"/>
+  <xacro:arg name="kinematics_params" default="$(find ur_description)/config/$(arg ur_type)/default_kinematics.yaml"/>
+  <xacro:arg name="physical_params" default="$(find ur_description)/config/$(arg ur_type)/physical_parameters.yaml"/>
+  <xacro:arg name="visual_params" default="$(find ur_description)/config/$(arg ur_type)/visual_parameters.yaml"/>
+  <xacro:arg name="use_fake_hardware" default="true" />
+  <xacro:arg name="fake_sensor_commands" default="true" />
+  <xacro:arg name="sim_gazebo" default="false" />
+  <xacro:arg name="sim_ignition" default="false" />
+  <xacro:arg name="robot_ip" default="192.168.0.210" />
+  <xacro:include filename="$(find robot_description)/urdf/arms/ur/ur.urdf.xacro"/>
   <!-- Import all available sensors -->
   <xacro:include filename="$(find robotnik_sensors)/urdf/all_sensors.urdf.xacro" />
@@ -32,10 +48,6 @@
   <xacro:property name="gps_offset_y" value="-0.167"/>
   <xacro:property name="gps_offset_z" value="0.302"/>
-  <!-- Launch Arguments -->
-  <xacro:arg name="use_gazebo_classic" default="false" />
-  <xacro:arg name="use_gazebo_ignition" default="false" />
-  <xacro:arg name="gpu" default="true" />
-  <xacro:arg name="namespace" default="robot" />
   <xacro:rbkairos/>
+  <!-- <xacro:include filename="$(find robot_description)/urdf/ros2_control/rbkairos_control.urdf.xacro" /> -->
   <!-- IMU -->
 	<xacro:sensor_vectornav prefix="rbkairos_" parent="rbkairos_base_link" topic="imu/data">

File: robot_description_simulation/ros2_control/classic/rbkairos_control.urdf.xacro (robot description, xacro)
@@ -6,5 +6,5 @@
             <robot_param>robot_description</robot_param>
             <robot_param_node>robot_state_publisher</robot_param_node>
-            <parameters>$(find robotnik_controller)/config/rbkairos_controller_example_params.yaml</parameters>
+            <parameters>$(find robotnik_gazebo_classic)/config/rbkairos_controller_params.yaml</parameters>
             <ros>
                 <namespace>/${namespace}</namespace>
@@ -33,22 +33,16 @@
         </ros2_control>
     </xacro:macro>
-    <xacro:macro name="ros_planar_move">
+    <xacro:macro name="ros_planar_move_gazebo">
         <gazebo>
           <plugin name="planar_move" filename="libgazebo_ros_planar_move.so">
             <ros>
               <!-- Remap the default topic -->
-              <remapping>cmd_vel:=cmd_vel_limited</remapping>
-              <remapping>odom:=rbkairos_odom</remapping>
+              <remapping>cmd_vel:=/robot/robotnik_base_controller/cmd_vel</remapping>
             </ros>
             <update_rate>100</update_rate>
             <publish_rate>10</publish_rate>
             <!-- output -->
-            <publish_odom>true</publish_odom>
-            <publish_odom_tf>true</publish_odom_tf>
-            <odometry_frame>rbkairos_odom</odometry_frame>
-            <robot_base_frame>rbkairos_base_link</robot_base_frame>
-            <covariance_x>0.0001</covariance_x>
-            <covariance_y>0.0001</covariance_y>
-            <covariance_yaw>0.01</covariance_yaw>
+            <publish_odom>false</publish_odom>
+            <publish_odom_tf>false</publish_odom_tf>
           </plugin>
         </gazebo>

File: robot_description_simulation/ros2_control/classic/rbsummit_control.urdf.xacro (robot description, xacro)
@@ -6,5 +6,5 @@
             <robot_param>robot_description</robot_param>
             <robot_param_node>robot_state_publisher</robot_param_node>
-            <parameters>$(find robotnik_controller)/config/rbsummit_controller_example_params.yaml</parameters>
+            <parameters>$(find robotnik_gazebo_classic)/config/rbsummit_controller_params.yaml</parameters>
             <ros>
                 <namespace>/${namespace}</namespace>

File: robot_description_simulation/ros2_control/classic/rbtheron_control.urdf.xacro (robot description, xacro)
@@ -6,5 +6,5 @@
             <robot_param>robot_description</robot_param>
             <robot_param_node>robot_state_publisher</robot_param_node>
-            <parameters>$(find robotnik_controller)/config/rbtheron_controller_example_params.yaml</parameters>
+            <parameters>$(find robotnik_gazebo_classic)/config/rbtheron_controller_params.yaml</parameters>
             <ros>
                 <namespace>/${namespace}</namespace>

File: robot_description_simulation/ros2_control/classic/rbvogui_control.urdf.xacro (robot description, xacro)
@@ -6,5 +6,5 @@
             <robot_param>robot_description</robot_param>
             <robot_param_node>robot_state_publisher</robot_param_node>
-            <parameters>$(find robotnik_controller)/config/rbvogui_controller_example_params.yaml</parameters>
+            <parameters>$(find robotnik_gazebo_classic)/config/rbvogui_controller_params.yaml</parameters>
             <ros>
                 <namespace>/${namespace}</namespace>

File: robot_description_simulation/ros2_control/ignition/rbkairos_control.urdf.xacro (robot description, xacro)
@@ -33,22 +33,16 @@
         </ros2_control>
     </xacro:macro>
-    <xacro:macro name="ros_planar_move">
+    <xacro:macro name="ros_planar_move_ignition">
         <gazebo>
           <plugin name="planar_move" filename="libgazebo_ros_planar_move.so">
             <ros>
               <!-- Remap the default topic -->
-              <remapping>cmd_vel:=cmd_vel_limited</remapping>
-              <remapping>odom:=rbkairos_odom</remapping>
+              <remapping>cmd_vel:=/robot/robotnik_base_controller/cmd_vel</remapping>
             </ros>
             <update_rate>100</update_rate>
             <publish_rate>10</publish_rate>
             <!-- output -->
-            <publish_odom>true</publish_odom>
-            <publish_odom_tf>true</publish_odom_tf>
-            <odometry_frame>rbkairos_odom</odometry_frame>
-            <robot_base_frame>rbkairos_base_link</robot_base_frame>
-            <covariance_x>0.0001</covariance_x>
-            <covariance_y>0.0001</covariance_y>
-            <covariance_yaw>0.01</covariance_yaw>
+            <publish_odom>false</publish_odom>
+            <publish_odom_tf>false</publish_odom_tf>
           </plugin>
         </gazebo>
