Commit message: update robot_description_simulation readme

File: robot_description_simulation/robots/rbkairos/rbkairos.urdf.xacro (robot description, xacro)
@@ -5,5 +5,5 @@
   <!-- ***************** -->
   <!-- First we import all posible elements defined in the urdf.xacro files. All these elements are defined as macro:xacros -->
-  <xacro:include filename="$(find robot_description)/macros/rbkairos_macro.urdf.xacro" />
+  <xacro:include filename="$(find robot_description)/bases/rbkairos/rbkairos_base.urdf.xacro" />
   <xacro:include filename="$(find robot_description_simulation)/ros2_control/classic/rbkairos_control.urdf.xacro"/>
   <xacro:include filename="$(find robot_description_simulation)/ros2_control/ignition/rbkairos_control.urdf.xacro"/>
@@ -39,14 +39,14 @@
   <xacro:rbkairos/>
   <!-- IMU -->
-	<xacro:sensor_vectornav prefix="rbkairos_" parent="rbkairos_base_link" topic="imu/data">
+	<!-- <xacro:sensor_vectornav prefix="rbkairos_" parent="rbkairos_base_link" topic="imu/data">
     <origin xyz="${imu_offset_x} ${imu_offset_y} ${imu_offset_z}" rpy="0 0 0"/>
-  </xacro:sensor_vectornav>
+  </xacro:sensor_vectornav> -->
   <!-- SENSORS -->
-  <xacro:sensor_sick_s300 prefix="rbkairos_front_laser" parent="rbkairos_base_link" prefix_topic="front_laser" gpu="true">
+  <!-- <xacro:sensor_sick_s300 prefix="rbkairos_front_laser" parent="rbkairos_base_link" prefix_topic="front_laser" gpu="true">
     <origin xyz="${front_laser_offset_x} ${front_laser_offset_y} ${front_laser_offset_z}" rpy="0 ${-PI} ${3/4*PI}" />
   </xacro:sensor_sick_s300>
   <xacro:sensor_sick_s300 prefix="rbkairos_rear_laser" parent="rbkairos_base_link" prefix_topic="rear_laser" gpu="true">
     <origin xyz="${rear_laser_offset_x} ${rear_laser_offset_y} ${rear_laser_offset_z}" rpy="0 ${-PI} ${-1/4*PI}" />
-  </xacro:sensor_sick_s300>
+  </xacro:sensor_sick_s300> -->
   <!--xacro:sensor_axis_m5013 prefix="$(arg prefix)front_ptz_camera" parent="$(arg prefix)base_link">
     <origin xyz="${front_ptz_camera_offset_x} ${front_ptz_camera_offset_y} ${front_ptz_camera_offset_z}" rpy="${-PI/2} 0 0"/>

File: robot_description_simulation/robots/rbkairos/rbkairos_ur.urdf.xacro (robot description, xacro)
@@ -6,5 +6,5 @@
   <!-- First we import all posible elements defined in the urdf.xacro files. All these elements are defined as macro:xacros -->
   <xacro:arg name="controllers" default="$(find robotnik_gazebo_classic)/config/rbkairos_control_gazebo.yaml"/>
-  <xacro:include filename="$(find robot_description)/macros/rbkairos_macro.urdf.xacro" />
+  <xacro:include filename="$(find robot_description)/bases/rbkairos/rbkairos_base.urdf.xacro" />
   <xacro:include filename="$(find robot_description_simulation)/ros2_control/classic/rbkairos_control.urdf.xacro"/>
   <xacro:include filename="$(find robot_description_simulation)/ros2_control/ignition/rbkairos_control.urdf.xacro"/>
@@ -51,26 +51,14 @@
   <!-- <xacro:include filename="$(find robot_description)/urdf/ros2_control/rbkairos_control.urdf.xacro" /> -->
   <!-- IMU -->
-	<xacro:sensor_vectornav prefix="rbkairos_" parent="rbkairos_base_link" topic="imu/data">
+	<!-- <xacro:sensor_vectornav prefix="rbkairos_" parent="rbkairos_base_link" topic="imu/data">
     <origin xyz="${imu_offset_x} ${imu_offset_y} ${imu_offset_z}" rpy="0 0 0"/>
-  </xacro:sensor_vectornav>
+  </xacro:sensor_vectornav> -->
   <!-- SENSORS -->
-  <xacro:sensor_sick_s300 prefix="rbkairos_front_laser" parent="rbkairos_base_link" prefix_topic="front_laser" gpu="true">
+  <!-- <xacro:sensor_sick_s300 prefix="rbkairos_front_laser" parent="rbkairos_base_link" prefix_topic="front_laser" gpu="true">
     <origin xyz="${front_laser_offset_x} ${front_laser_offset_y} ${front_laser_offset_z}" rpy="0 ${-PI} ${3/4*PI}" />
   </xacro:sensor_sick_s300>
   <xacro:sensor_sick_s300 prefix="rbkairos_rear_laser" parent="rbkairos_base_link" prefix_topic="rear_laser" gpu="true">
     <origin xyz="${rear_laser_offset_x} ${rear_laser_offset_y} ${rear_laser_offset_z}" rpy="0 ${-PI} ${-1/4*PI}" />
-  </xacro:sensor_sick_s300>
-  <!--xacro:sensor_axis_m5013 prefix="$(arg prefix)front_ptz_camera" parent="$(arg prefix)base_link">
-    <origin xyz="${front_ptz_camera_offset_x} ${front_ptz_camera_offset_y} ${front_ptz_camera_offset_z}" rpy="${-PI/2} 0 0"/>
-  </xacro:sensor_axis_m5013-->
-  <!--xacro:sensor_axis_m5013 prefix="$(arg prefix)rear_ptz_camera" parent="$(arg prefix)base_link">
-    <origin xyz="${rear_ptz_camera_offset_x} ${rear_ptz_camera_offset_y} ${rear_ptz_camera_offset_z}" rpy="${-PI/2} 0 ${PI}"/>
-  </xacro:sensor_axis_m5013-->
-  <!-- <xacro:sensor_orbbec_astra prefix="$(arg prefix)front_rgbd_camera" parent="$(arg prefix)base_link" prefix_topic="front_rgbd_camera">
-    <origin xyz="${front_rgbd_camera_offset_x} ${front_rgbd_camera_offset_y} ${front_rgbd_camera_offset_z}" rpy="0 0 0"/>
-  </xacro:sensor_orbbec_astra> -->
-  <!--xacro:sensor_gps prefix="$(arg prefix)gps" parent="$(arg prefix)base_link">
-    <origin xyz="${gps_offset_x} ${gps_offset_y} ${gps_offset_z}" rpy="0 0 0"/>
-  </xacro:sensor_gps-->
+  </xacro:sensor_sick_s300> -->
   <xacro:if value="$(arg use_gazebo_classic)">
       <xacro:rbkairos_gz_classic_control namespace="$(arg namespace)"/>

File: robot_description_simulation/robots/rbsteel/rbsteel.urdf.xacro (robot description, xacro)
@@ -6,5 +6,5 @@
   <!-- First we import all posible elements defined in the urdf.xacro files. All these elements are defined as macro:xacros -->
   <xacro:arg name="controllers" default="$(find robot_gazebo)/config/rbkairos_control_gazebo.yaml"/>
-  <xacro:include filename="$(find robot_description)/robots/macros/rbsteel_macro.urdf.xacro" />
+  <xacro:include filename="$(find robot_description)/bases/rbsteel/rbsteel_base.urdf.xacro" />
   <!-- Import all available sensors -->
   <xacro:include filename="$(find robotnik_sensors)/urdf/all_sensors.urdf.xacro" />
@@ -32,16 +32,15 @@
   <xacro:property name="gps_offset_z" value="0.302"/>
   <xacro:rbkairos/>
-  <xacro:include filename="$(find robot_description)/urdf/ros2_control/rbkairos_control.urdf.xacro" />
   <!-- IMU -->
-	<xacro:sensor_vectornav prefix="rbkairos_" parent="rbkairos_base_link" topic="imu/data">
+	<!-- <xacro:sensor_vectornav prefix="rbkairos_" parent="rbkairos_base_link" topic="imu/data">
     <origin xyz="${imu_offset_x} ${imu_offset_y} ${imu_offset_z}" rpy="0 0 0"/>
-  </xacro:sensor_vectornav>
+  </xacro:sensor_vectornav> -->
   <!-- SENSORS -->
-  <xacro:sensor_sick_s300 prefix="rbkairos_front_laser" parent="rbkairos_base_link" prefix_topic="front_laser" gpu="true">
+  <!-- <xacro:sensor_sick_s300 prefix="rbkairos_front_laser" parent="rbkairos_base_link" prefix_topic="front_laser" gpu="true">
     <origin xyz="${front_laser_offset_x} ${front_laser_offset_y} ${front_laser_offset_z}" rpy="0 ${-PI} ${3/4*PI}" />
   </xacro:sensor_sick_s300>
   <xacro:sensor_sick_s300 prefix="rbkairos_rear_laser" parent="rbkairos_base_link" prefix_topic="rear_laser" gpu="true">
     <origin xyz="${rear_laser_offset_x} ${rear_laser_offset_y} ${rear_laser_offset_z}" rpy="0 ${-PI} ${-1/4*PI}" />
-  </xacro:sensor_sick_s300>
+  </xacro:sensor_sick_s300> -->
   <!--xacro:sensor_axis_m5013 prefix="$(arg prefix)front_ptz_camera" parent="$(arg prefix)base_link">
     <origin xyz="${front_ptz_camera_offset_x} ${front_ptz_camera_offset_y} ${front_ptz_camera_offset_z}" rpy="${-PI/2} 0 0"/>

File: robot_description_simulation/robots/rbsummit/rbsummit.urdf.xacro (robot description, xacro)
@@ -6,5 +6,5 @@
 	<!-- First we import the robot and all the sensors. All these elements are defined as macro:xacros -->
 	<!-- Import summit XL macro -->
-	<xacro:include filename="$(find robot_description)/macros/rbsummit_macro.xacro"/>
+	<xacro:include filename="$(find robot_description)/bases/rbsummit/rbsummit_base.xacro"/>
 	<!-- Import all available sensors -->
 	<xacro:include filename="$(find robotnik_sensors)/urdf/all_sensors.urdf.xacro" />
@@ -31,7 +31,7 @@
 	<!-- Custom Sensors -->
 	<!-- IMU -->
-	<xacro:sensor_vectornav prefix="rbsummit_" parent="rbsummit_base_link" topic="imu/data">
+	<!-- <xacro:sensor_vectornav prefix="rbsummit_" parent="rbsummit_base_link" topic="imu/data">
 		<origin xyz="0.0385 0.132 0.158" rpy="0 0 0"/>
-  </xacro:sensor_vectornav>
+  </xacro:sensor_vectornav> -->
 	<!-- 3d laser -->
 	<!-- <xacro:sensor_rs_helios_16p prefix="$(arg prefix)top_3d_laser" parent="$(arg prefix)base_link" gpu="$(arg gpu)">

File: robot_description_simulation/robots/rbtheron/rbtheron.urdf.xacro (robot description, xacro)
@@ -7,5 +7,5 @@
 	<!-- First we import all posible elements defined in the urdf.xacro files. All these elements are defined as macro:xacros -->
 	<!-- Import rbtheron macro -->
-	<xacro:include filename="$(find robot_description)/macros/rbtheron_macro.xacro"/>
+	<xacro:include filename="$(find robot_description)/bases/rbtheron/rbtheron_base.xacro"/>
 	<!-- Import all available sensors -->
 	<xacro:include filename="$(find robotnik_sensors)/urdf/all_sensors.urdf.xacro" />
@@ -35,13 +35,13 @@
 	<xacro:rbtheron hq="${hq}"/>
 	<!-- ELEVATOR_PLATFORM -->
-	<xacro:if value="$(arg has_elevator)">
+	<!-- <xacro:if value="$(arg has_elevator)">
 		<xacro:elevator_platform robot_id="rbtheron_elevator" parent="rbtheron_base_link" hq="${hq}">
 			<origin xyz="${elevator_x} -${elevator_y} ${elevator_z}" rpy="1.5708 0 1.5708"/>
 		</xacro:elevator_platform>
-	</xacro:if>
+	</xacro:if> -->
 	<!-- SENSORS -->
-	<xacro:sensor_vectornav prefix="rbtheron_" parent="rbtheron_base_link" topic="imu/data">
+	<!-- <xacro:sensor_vectornav prefix="rbtheron_" parent="rbtheron_base_link" topic="imu/data">
 		<origin xyz="-0.1975 0.0 0.1598" rpy="0 0 0"/>
-    </xacro:sensor_vectornav>
+    </xacro:sensor_vectornav> -->
     <xacro:if value="$(arg use_gazebo_classic)">
         <xacro:rbtheron_gz_classic_control namespace="$(arg namespace)"/>

File: robot_description_simulation/robots/rbvogui/rbvogui.urdf.xacro (robot description, xacro)
@@ -7,5 +7,5 @@
     <!-- First we import all posible elements defined in the urdf.xacro files. All these elements are defined as macro:xacros -->
     <!-- Import rbvogui base elements-->
-    <xacro:include filename="$(find robot_description)/macros/rbvogui_macro.urdf.xacro" />
+    <xacro:include filename="$(find robot_description)/bases/rbvogui/rbvogui_base.urdf.xacro" />
     <xacro:include filename="$(find robot_description_simulation)/ros2_control/classic/rbvogui_control.urdf.xacro"/>
     <xacro:include filename="$(find robot_description_simulation)/ros2_control/ignition/rbvogui_control.urdf.xacro"/>
@@ -23,22 +23,22 @@
     <!-- SENSORS see robotnik_sensors for the specific configuration -->
     <!-- IMU -->
-    <xacro:sensor_vectornav prefix="rbvogui_" parent="rbvogui_chassis_link" topic="imu/data">
+    <!-- <xacro:sensor_vectornav prefix="rbvogui_" parent="rbvogui_chassis_link" topic="imu/data">
         <origin xyz="0.3 -0.3 0.0725" rpy="0 0 0"/>
-    </xacro:sensor_vectornav>
+    </xacro:sensor_vectornav> -->
     <!-- Front Camera -->
-    <xacro:sensor_intel_d435 prefix="rbvogui_front_rgbd_camera" parent="rbvogui_chassis_link" prefix_topic="front_rgbd_camera" use_nominal_extrinsics="true">
+    <!-- <xacro:sensor_intel_d435 prefix="rbvogui_front_rgbd_camera" parent="rbvogui_chassis_link" prefix_topic="front_rgbd_camera" use_nominal_extrinsics="true">
         <origin xyz="0.46462 0.0 0.18258" rpy="0 0 0"/>
-    </xacro:sensor_intel_d435>
+    </xacro:sensor_intel_d435> -->
     <!-- Rear Camera -->
-    <xacro:sensor_intel_d435 prefix="rbvogui_rear_rgbd_camera" parent="rbvogui_base_link" prefix_topic="rear_rgbd_camera" use_nominal_extrinsics="true">
+    <!-- <xacro:sensor_intel_d435 prefix="rbvogui_rear_rgbd_camera" parent="rbvogui_base_link" prefix_topic="rear_rgbd_camera" use_nominal_extrinsics="true">
         <origin xyz="-0.503 0.0 0.29" rpy="0 0 -${PI}"/>
-    </xacro:sensor_intel_d435>
+    </xacro:sensor_intel_d435> -->
     <!-- 2d laser -->
-    <xacro:sensor_sick_s300 prefix="rbvogui_front_laser" parent="rbvogui_chassis_link" gpu="$(arg gpu)" prefix_topic="front_laser">
+    <!-- <xacro:sensor_sick_s300 prefix="rbvogui_front_laser" parent="rbvogui_chassis_link" gpu="$(arg gpu)" prefix_topic="front_laser">
         <origin xyz="0.53 0.33 0.1145" rpy="${PI} 0 ${PI/4}"/>
     </xacro:sensor_sick_s300>
     <xacro:sensor_sick_s300 prefix="rbvogui_rear_laser" parent="rbvogui_chassis_link" gpu="$(arg gpu)" prefix_topic="rear_laser">
         <origin xyz="-0.53 -0.33 0.1145" rpy="${PI} 0 ${-PI*3/4}"/>
-    </xacro:sensor_sick_s300>
+    </xacro:sensor_sick_s300> -->
     <xacro:if value="$(arg use_gazebo_classic)">
         <xacro:rbvogui_gz_classic_control namespace="$(arg namespace)"/>

File: robot_description_simulation/robots/rbvogui/rbvogui_cart.urdf.xacro (robot description, xacro)
@@ -7,5 +7,5 @@
     <!-- First we import all posible elements defined in the urdf.xacro files. All these elements are defined as macro:xacros -->
     <!-- Import rbvogui base elements-->
-    <xacro:include filename="$(find robot_description)/robots/macros/rbvogui_macro.urdf.xacro" />
+    <xacro:include filename="$(find robot_description)/bases/rbvogui/rbvogui_base.urdf.xacro" />
     <xacro:include filename="$(find robot_description)/urdf/ros2_control/rbvogui_control.urdf.xacro"/>
     <!-- Import all available sensors -->
